Commit message: added PandaArm urdf, robot class

File: jkinpylib/urdfs/panda_arm/panda_arm_hand.urdf (robot description, URDF)
Before this commit: robot panda, 12 links, 11 joints
Links:
- link panda_hand: mass None -> 0.67893; geometry collision mesh filename=package://panda_description/meshes/collision/hand.stl; visual mesh filename=package://panda_description/meshes/visual/hand.dae
- link panda_leftfinger: mass None -> 0.01053; geometry collision mesh filename=package://panda_description/meshes/collision/finger.stl; visual mesh filename=package://panda_description/meshes/visual/finger.dae
- link panda_link0: mass None -> 4; geometry collision mesh filename=package://panda_description/meshes/collision/link0.stl; visual mesh filename=package://panda_description/meshes/visual/link0.dae
- link panda_link1: mass None -> 3; geometry collision mesh filename=package://panda_description/meshes/collision/link1.stl; visual mesh filename=package://panda_description/meshes/visual/link1.dae
- link panda_link2: mass None -> 3; geometry collision mesh filename=package://panda_description/meshes/collision/link2.stl; visual mesh filename=package://panda_description/meshes/visual/link2.dae
- link panda_link3: mass None -> 2; geometry collision mesh filename=package://panda_description/meshes/collision/link3.stl; visual mesh filename=package://panda_description/meshes/visual/link3.dae
- link panda_link4: mass None -> 2; geometry collision mesh filename=package://panda_description/meshes/collision/link4.stl; visual mesh filename=package://panda_description/meshes/visual/link4.dae
- link panda_link5: mass None -> 2; geometry collision mesh filename=package://panda_description/meshes/collision/link5.stl; visual mesh filename=package://panda_description/meshes/visual/link5.dae
- link panda_link6: mass None -> 1.5; geometry collision mesh filename=package://panda_description/meshes/collision/link6.stl; visual mesh filename=package://panda_description/meshes/visual/link6.dae
- link panda_link7: mass None -> 0.5; geometry collision mesh filename=package://panda_description/meshes/collision/link7.stl; visual mesh filename=package://panda_description/meshes/visual/link7.dae
- link panda_link8: mass None -> 0.005
- link panda_rightfinger: mass None -> 0.01053; geometry collision mesh filename=package://panda_description/meshes/collision/finger.stl; visual mesh filename=package://panda_description/meshes/visual/finger.dae
Joints:
- joint panda_joint1: limit lower=-2.9671 upper=2.9671 effort=87 velocity=2.1750 -> lower=-2.8973 upper=2.8973 effort=87 velocity=2.1750; origin xyz=0 0 0.333 rpy=0 0 0 -> xyz=0 -0.1 0 rpy=0 0 0
- joint panda_joint2: limit lower=-1.8326 upper=1.8326 effort=87 velocity=2.1750 -> lower=-1.7628 upper=1.7628 effort=87 velocity=2.1750
- joint panda_joint3: limit lower=-2.9671 upper=2.9671 effort=87 velocity=2.1750 -> lower=-2.8973 upper=2.8973 effort=87 velocity=2.1750
- joint panda_joint4: limit lower=-3.1416 upper=0.0 effort=87 velocity=2.1750 -> lower=-3.0718 upper=-0.0698 effort=87 velocity=2.1750
- joint panda_joint5: limit lower=-2.9671 upper=2.9671 effort=12 velocity=2.6100 -> lower=-2.8973 upper=2.8973 effort=12 velocity=2.6100
- joint panda_joint6: limit lower=-0.0873 upper=3.8223 effort=12 velocity=2.6100 -> lower=-0.0175 upper=3.7525 effort=12 velocity=2.6100
- joint panda_joint7: limit lower=-2.9671 upper=2.9671 effort=12 velocity=2.6100 -> lower=-2.8973 upper=2.8973 effort=12 velocity=2.6100

File: jkinpylib/urdfs/panda_arm/panda_arm_hand_formatted.urdf (robot description, URDF)
Before this commit: robot panda, 12 links, 11 joints
Links:
- link panda_hand: mass None -> 0.67893; geometry collision mesh filename=meshes/collision/hand.stl; visual mesh filename=meshes/visual/hand.dae
- link panda_leftfinger: mass None -> 0.01053; geometry collision mesh filename=meshes/collision/finger.stl; visual mesh filename=meshes/visual/finger.dae
- link panda_link0: mass None -> 4; geometry collision mesh filename=meshes/collision/link0.stl; visual mesh filename=meshes/visual/link0.dae
- link panda_link1: mass None -> 3; geometry collision mesh filename=meshes/collision/link1.stl; visual mesh filename=meshes/visual/link1.dae
- link panda_link2: mass None -> 3; geometry collision mesh filename=meshes/collision/link2.stl; visual mesh filename=meshes/visual/link2.dae
- link panda_link3: mass None -> 2; geometry collision mesh filename=meshes/collision/link3.stl; visual mesh filename=meshes/visual/link3.dae
- link panda_link4: mass None -> 2; geometry collision mesh filename=meshes/collision/link4.stl; visual mesh filename=meshes/visual/link4.dae
- link panda_link5: mass None -> 2; geometry collision mesh filename=meshes/collision/link5.stl; visual mesh filename=meshes/visual/link5.dae
- link panda_link6: mass None -> 1.5; geometry collision mesh filename=meshes/collision/link6.stl; visual mesh filename=meshes/visual/link6.dae
- link panda_link7: mass None -> 0.5; geometry collision mesh filename=meshes/collision/link7.stl; visual mesh filename=meshes/visual/link7.dae
- link panda_link8: mass None -> 0.005
- link panda_rightfinger: mass None -> 0.01053; geometry collision mesh filename=meshes/collision/finger.stl; visual mesh filename=meshes/visual/finger.dae
Joints:
- joint panda_joint1: limit lower=-2.9671 upper=2.9671 effort=87 velocity=2.1750 -> lower=-2.8973 upper=2.8973 effort=87 velocity=2.1750
- joint panda_joint2: limit lower=-1.8326 upper=1.8326 effort=87 velocity=2.1750 -> lower=-1.7628 upper=1.7628 effort=87 velocity=2.1750
- joint panda_joint3: limit lower=-2.9671 upper=2.9671 effort=87 velocity=2.1750 -> lower=-2.8973 upper=2.8973 effort=87 velocity=2.1750
- joint panda_joint4: limit lower=-3.1416 upper=0.0 effort=87 velocity=2.1750 -> lower=-3.0718 upper=-0.0698 effort=87 velocity=2.1750
- joint panda_joint5: limit lower=-2.9671 upper=2.9671 effort=12 velocity=2.6100 -> lower=-2.8973 upper=2.8973 effort=12 velocity=2.6100
- joint panda_joint6: limit lower=-0.0873 upper=3.8223 effort=12 velocity=2.6100 -> lower=-0.0175 upper=3.7525 effort=12 velocity=2.6100
- joint panda_joint7: limit lower=-2.9671 upper=2.9671 effort=12 velocity=2.6100 -> lower=-2.8973 upper=2.8973 effort=12 velocity=2.6100
