Commit message: added get_urdf_filepath_w_filenames_updated()

File: jkinpylib/urdfs/baxter/baxter.urdf (robot description, URDF)
Before this commit: robot baxter, 57 links, 56 joints
Links:
- link head: geometry collision sphere radius=0.001; visual mesh filename=urdfs/baxter/meshes/head/H0.STL
- link l_gripper_l_finger: geometry collision box size=0.01 0.0135 0.1127; collision box size=0.01 0.05 0.017
- link l_gripper_l_finger_tip: geometry collision box size=0.042 0.0065 0.037; visual mesh filename=urdfs/baxter/meshes/electric_gripper/fingers/paddle_tip.STL
- link l_gripper_r_finger: geometry collision box size=0.01 0.0135 0.1127; collision box size=0.01 0.05 0.017
- link l_gripper_r_finger_tip: geometry collision box size=0.042 0.0065 0.037; visual mesh filename=urdfs/baxter/meshes/electric_gripper/fingers/paddle_tip.STL
- link left_gripper_base: geometry collision cylinder length=0.1 radius=0.029; visual mesh filename=urdfs/baxter/meshes/electric_gripper/electric_gripper_base.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
- link left_lower_elbow: geometry collision cylinder length=0.10 radius=0.06; visual mesh filename=urdfs/baxter/meshes/lower_elbow/E1.STL
- link left_lower_forearm: geometry collision cylinder length=0.10 radius=0.06; visual mesh filename=urdfs/baxter/meshes/lower_forearm/W1.STL
- link left_lower_shoulder: geometry collision cylinder length=0.12 radius=0.06; visual mesh filename=urdfs/baxter/meshes/lower_shoulder/S1.STL
- link left_upper_elbow: geometry collision cylinder length=0.107 radius=0.06; visual mesh filename=urdfs/baxter/meshes/upper_elbow/E0.STL
- link left_upper_forearm: geometry collision cylinder length=0.088 radius=0.06; visual mesh filename=urdfs/baxter/meshes/upper_forearm/W0.STL
- link left_upper_shoulder: geometry collision cylinder length=0.2722 radius=0.06; visual mesh filename=urdfs/baxter/meshes/upper_shoulder/S0.STL
- link left_wrist: geometry collision cylinder length=0.165 radius=0.06; visual mesh filename=urdfs/baxter/meshes/wrist/W2.STL
- link pedestal: geometry collision mesh filename=urdfs/baxter/meshes/base/pedestal_link_collision.STL; visual mesh filename=urdfs/baxter/meshes/base/PEDESTAL.STL
- link r_gripper_l_finger: geometry collision box size=0.01 0.0135 0.1127; collision box size=0.01 0.05 0.017
- link r_gripper_l_finger_tip: geometry collision cylinder length=0.037 radius=0.008; visual mesh filename=urdfs/baxter/meshes/electric_gripper/fingers/half_round_tip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
- link r_gripper_r_finger: geometry collision box size=0.01 0.0135 0.1127; collision box size=0.01 0.05 0.017
- link r_gripper_r_finger_tip: geometry collision cylinder length=0.037 radius=0.008; visual mesh filename=urdfs/baxter/meshes/electric_gripper/fingers/half_round_tip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
- link right_gripper_base: geometry collision cylinder length=0.1 radius=0.029; visual mesh filename=urdfs/baxter/meshes/electric_gripper/electric_gripper_base.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
- link right_lower_elbow: geometry collision cylinder length=0.10 radius=0.06; visual mesh filename=urdfs/baxter/meshes/lower_elbow/E1.STL
- link right_lower_forearm: geometry collision cylinder length=0.10 radius=0.06; visual mesh filename=urdfs/baxter/meshes/lower_forearm/W1.STL
- link right_lower_shoulder: geometry collision cylinder length=0.12 radius=0.06; visual mesh filename=urdfs/baxter/meshes/lower_shoulder/S1.STL
- link right_upper_elbow: geometry collision cylinder length=0.107 radius=0.06; visual mesh filename=urdfs/baxter/meshes/upper_elbow/E0.STL
- link right_upper_forearm: geometry collision cylinder length=0.088 radius=0.06; visual mesh filename=urdfs/baxter/meshes/upper_forearm/W0.STL
- link right_upper_shoulder: geometry collision cylinder length=0.2722 radius=0.06; visual mesh filename=urdfs/baxter/meshes/upper_shoulder/S0.STL
- link right_wrist: geometry collision cylinder length=0.165 radius=0.06; visual mesh filename=urdfs/baxter/meshes/wrist/W2.STL
- link screen: geometry collision sphere radius=0.001; visual mesh filename=urdfs/baxter/meshes/head/H1.STL
- link torso: geometry collision mesh filename=urdfs/baxter/meshes/torso/base_link_collision.STL; visual mesh filename=urdfs/baxter/meshes/torso/base_link.STL

File: jkinpylib/urdfs/fetch/fetch_formatted.urdf (robot description, URDF)
Before this commit: robot fetch, 25 links, 24 joints
Links:
- link base_link: geometry collision cylinder length=0.33 radius=0.28; visual mesh filename=urdfs/fetch/meshes/base_link.dae
- link bellows_link2: geometry collision mesh filename=urdfs/fetch/meshes/bellows_link_collision.STL; visual mesh filename=urdfs/fetch/meshes/bellows_link.STL
- link elbow_flex_link: geometry collision mesh filename=urdfs/fetch/meshes/elbow_flex_link_collision.STL; visual mesh filename=urdfs/fetch/meshes/elbow_flex_link.dae
- link estop_link: geometry collision mesh filename=urdfs/fetch/meshes/estop_link.STL; visual mesh filename=urdfs/fetch/meshes/estop_link.STL
- link forearm_roll_link: geometry collision mesh filename=urdfs/fetch/meshes/forearm_roll_link_collision.STL; visual mesh filename=urdfs/fetch/meshes/forearm_roll_link.dae
- link gripper_link: geometry collision mesh filename=urdfs/fetch/meshes/gripper_link.STL; visual mesh filename=urdfs/fetch/meshes/gripper_link.dae
- link head_pan_link: geometry collision mesh filename=urdfs/fetch/meshes/head_pan_link_collision.STL; visual mesh filename=urdfs/fetch/meshes/head_pan_link.dae
- link head_tilt_link: geometry collision mesh filename=urdfs/fetch/meshes/head_tilt_link_collision.STL; visual mesh filename=urdfs/fetch/meshes/head_tilt_link.dae
- link l_gripper_finger_link: geometry collision box size=0.062 0.013 0.026; visual mesh filename=urdfs/fetch/meshes/l_gripper_finger_link.STL
- link l_wheel_link: geometry collision sphere radius=0.065; visual mesh filename=urdfs/fetch/meshes/l_wheel_link.STL
- link laser_link: geometry collision mesh filename=urdfs/fetch/meshes/laser_link.STL; visual mesh filename=urdfs/fetch/meshes/laser_link.STL
- link r_gripper_finger_link: geometry collision box size=0.062 0.013 0.026; visual mesh filename=urdfs/fetch/meshes/r_gripper_finger_link.STL
- link r_wheel_link: geometry collision sphere radius=0.065; visual mesh filename=urdfs/fetch/meshes/r_wheel_link.STL
- link shoulder_lift_link: geometry collision mesh filename=urdfs/fetch/meshes/shoulder_lift_link_collision.STL; visual mesh filename=urdfs/fetch/meshes/shoulder_lift_link.dae
- link shoulder_pan_link: geometry collision mesh filename=urdfs/fetch/meshes/shoulder_pan_link_collision.STL; visual mesh filename=urdfs/fetch/meshes/shoulder_pan_link.dae
- link torso_fixed_link: geometry collision mesh filename=urdfs/fetch/meshes/torso_fixed_link.STL; visual mesh filename=urdfs/fetch/meshes/torso_fixed_link.dae
- link torso_lift_link: geometry collision mesh filename=urdfs/fetch/meshes/torso_lift_link_collision.STL; visual mesh filename=urdfs/fetch/meshes/torso_lift_link.dae
- link upperarm_roll_link: geometry collision mesh filename=urdfs/fetch/meshes/upperarm_roll_link_collision.STL; visual mesh filename=urdfs/fetch/meshes/upperarm_roll_link.dae
- link wrist_flex_link: geometry collision mesh filename=urdfs/fetch/meshes/wrist_flex_link_collision.STL; visual mesh filename=urdfs/fetch/meshes/wrist_flex_link.dae
- link wrist_roll_link: geometry collision mesh filename=urdfs/fetch/meshes/wrist_roll_link_collision.STL; visual mesh filename=urdfs/fetch/meshes/wrist_roll_link.dae

File: jkinpylib/urdfs/iiwa7/iiwa7_formatted.urdf (robot description, URDF)
Before this commit: robot iiwa7, 10 links, 9 joints
Links:
- link iiwa_link_0: geometry collision mesh filename=urdfs/iiwa7/meshes/collision/link_0.stl; visual mesh filename=urdfs/iiwa7/meshes/visual/link_0.stl
- link iiwa_link_1: geometry collision mesh filename=urdfs/iiwa7/meshes/collision/link_1.stl; visual mesh filename=urdfs/iiwa7/meshes/visual/link_1.stl
- link iiwa_link_2: geometry collision mesh filename=urdfs/iiwa7/meshes/collision/link_2.stl; visual mesh filename=urdfs/iiwa7/meshes/visual/link_2.stl
- link iiwa_link_3: geometry collision mesh filename=urdfs/iiwa7/meshes/collision/link_3.stl; visual mesh filename=urdfs/iiwa7/meshes/visual/link_3.stl
- link iiwa_link_4: geometry collision mesh filename=urdfs/iiwa7/meshes/collision/link_4.stl; visual mesh filename=urdfs/iiwa7/meshes/visual/link_4.stl
- link iiwa_link_5: geometry collision mesh filename=urdfs/iiwa7/meshes/collision/link_5.stl; visual mesh filename=urdfs/iiwa7/meshes/visual/link_5.stl
- link iiwa_link_6: geometry collision mesh filename=urdfs/iiwa7/meshes/collision/link_6.stl; visual mesh filename=urdfs/iiwa7/meshes/visual/link_6.stl
- link iiwa_link_7: geometry collision mesh filename=urdfs/iiwa7/meshes/collision/link_7.stl; visual mesh filename=urdfs/iiwa7/meshes/visual/link_7.stl

File: jkinpylib/urdfs/panda/panda_arm_hand_formatted.urdf (robot description, URDF)
Before this commit: robot panda, 12 links, 11 joints
Links:
- link panda_hand: geometry collision mesh filename=urdfs/panda/meshes/collision/hand.stl; visual mesh filename=urdfs/panda/meshes/visual/hand.dae
- link panda_leftfinger: geometry collision mesh filename=urdfs/panda/meshes/collision/finger.stl; visual mesh filename=urdfs/panda/meshes/visual/finger.dae
- link panda_link0: geometry collision mesh filename=urdfs/panda/meshes/collision/link0.stl; visual mesh filename=urdfs/panda/meshes/visual/link0.dae
- link panda_link1: geometry collision mesh filename=urdfs/panda/meshes/collision/link1.stl; visual mesh filename=urdfs/panda/meshes/visual/link1.dae
- link panda_link2: geometry collision mesh filename=urdfs/panda/meshes/collision/link2.stl; visual mesh filename=urdfs/panda/meshes/visual/link2.dae
- link panda_link3: geometry collision mesh filename=urdfs/panda/meshes/collision/link3.stl; visual mesh filename=urdfs/panda/meshes/visual/link3.dae
- link panda_link4: geometry collision mesh filename=urdfs/panda/meshes/collision/link4.stl; visual mesh filename=urdfs/panda/meshes/visual/link4.dae
- link panda_link5: geometry collision mesh filename=urdfs/panda/meshes/collision/link5.stl; visual mesh filename=urdfs/panda/meshes/visual/link5.dae
- link panda_link6: geometry collision mesh filename=urdfs/panda/meshes/collision/link6.stl; visual mesh filename=urdfs/panda/meshes/visual/link6.dae
- link panda_link7: geometry collision mesh filename=urdfs/panda/meshes/collision/link7.stl; visual mesh filename=urdfs/panda/meshes/visual/link7.dae
- link panda_rightfinger: geometry collision mesh filename=urdfs/panda/meshes/collision/finger.stl; visual mesh filename=urdfs/panda/meshes/visual/finger.dae
