Commit message: adding repeatability code, added klampt tag to robot urdfs

File: jkinpylib/urdfs/fetch/fetch_formatted.urdf (robot description, URDF)
Before this commit: robot fetch, 25 links, 24 joints
Links:
- link l_gripper_finger_link: geometry collision box size=0.062 0.013 0.026; visual box size=0.062 0.013 0.026
- link r_gripper_finger_link: geometry collision box size=0.062 0.013 0.026; visual box size=0.062 0.013 0.026
