Commit message: modify velocity limit

File: jrl/urdfs/jaka/left_jaka.urdf (robot description, URDF)
Before this commit: robot jaka, 8 links, 7 joints
Joints:
- joint J_1: limit lower=-6.1927 upper=6.1927 effort=0 velocity=0 -> lower=-6.1927 upper=6.1927 effort=0 velocity=1.0
- joint J_2: limit lower=-1.6572 upper=1.6572 effort=0 velocity=0 -> lower=-1.6572 upper=1.6572 effort=0 velocity=1.0
- joint J_3: limit lower=-6.1927 upper=6.1927 effort=0 velocity=0 -> lower=-6.1927 upper=6.1927 effort=0 velocity=1.0
- joint J_4: limit lower=-2.2677 upper=0.3837 effort=0 velocity=0 -> lower=-2.2677 upper=0.3837 effort=0 velocity=1.0
- joint J_5: limit lower=-6.1927 upper=6.1927 effort=0 velocity=0 -> lower=-6.1927 upper=6.1927 effort=0 velocity=1.0
- joint J_6: limit lower=-1.5707 upper=1.5707 effort=0 velocity=0 -> lower=-1.5707 upper=1.5707 effort=0 velocity=1.0
- joint J_7: limit lower=-6.1927 upper=6.1927 effort=0 velocity=0 -> lower=-6.1927 upper=6.1927 effort=0 velocity=1.0

Commit message: modify meshes path

File: jrl/urdfs/jaka/left_jaka.urdf (robot description, URDF)
Before this commit: robot jaka, 8 links, 7 joints
Links:
- link LINK_1: geometry collision mesh filename=urdfs/jaka/meshes/LINK_1.STL; visual mesh filename=urdfs/jaka/meshes/LINK_1.STL
- link LINK_2: geometry collision mesh filename=urdfs/jaka/meshes/LINK_2.STL; visual mesh filename=urdfs/jaka/meshes/LINK_2.STL
- link LINK_3: geometry collision mesh filename=urdfs/jaka/meshes/LINK_3.STL; visual mesh filename=urdfs/jaka/meshes/LINK_3.STL
- link LINK_4: geometry collision mesh filename=urdfs/jaka/meshes/LINK_4.STL; visual mesh filename=urdfs/jaka/meshes/LINK_4.STL
- link LINK_5: geometry collision mesh filename=urdfs/jaka/meshes/LINK_5.STL; visual mesh filename=urdfs/jaka/meshes/LINK_5.STL
- link LINK_6: geometry collision mesh filename=urdfs/jaka/meshes/LINK_6.STL; visual mesh filename=urdfs/jaka/meshes/LINK_6.STL
- link LINK_7: geometry collision mesh filename=urdfs/jaka/meshes/LINK_7.STL; visual mesh filename=urdfs/jaka/meshes/LINK_7.STL
- link LINK_BASE: geometry collision mesh filename=urdfs/jaka/meshes/LINK_BASE.STL; visual mesh filename=urdfs/jaka/meshes/LINK_BASE.STL
