Commit message: added PandaHandTcp

File: jrl/urdfs/panda/panda_arm_hand_formatted.urdf (robot description, URDF)
Before this commit: robot panda, 12 links, 11 joints
Links:
- added link panda_hand_tcp
Joints:
- added joint panda_hand_tcp_joint: type fixed, parent panda_hand, child panda_hand_tcp, origin xyz=0 0 0.1034 rpy=0 0 0
